File: RatTrapSensorPCB.kicad_pcb (KiCad board)
At the start: 2 copper layers, 34.2 x 62.7 mm, 11 parts, among them U1 LoRaSx1276

Commit message: Corrected antenna output
Parts:
- added ?: , Pin_Headers:Pin_Header_Straight_1x02_Pitch2.54mm, F.Cu at (142.8, 160.7)
- moved ? 1.68 mm to (142.8, 157.3)
- gave numbers to parts that had none: 2
Connections:
- ? pad 1: ANT -> GND
- ? pad 2: GND -> ANT
Routing:
- net GND: track 94.1 -> 98.5 mm
- net ANT: track 11.7 -> 7.57 mm
Other:
- board text added: "v1.1 August 2018 D Q McDonald"
- board text removed: "v1.0 August 2018 D Q McDonald"
Changed lines of the file:
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@@
 (kicad_pcb (version 4) (host pcbnew 4.0.7)
   (general
-    (links 36)
+    (links 38)
     (no_connects 0)
-    (area 138.6 99.824999 176.33 162.700001)
+    (area 140.749999 99.824999 175.075001 162.700001)
     (thickness 1.6)
-    (drawings 26)
-    (tracks 139)
+    (drawings 27)
+    (tracks 141)
     (zones 0)
-    (modules 11)
+    (modules 12)
     (nets 30)
   )
@@
     (tags "resistor 0805")
     (attr smd)
-    (fp_text reference "" (at 0 -1.7 270) (layer F.SilkS)
+    (fp_text reference D1 (at 0 -1.7 270) (layer F.SilkS)
       (effects (font (size 1 1) (thickness 0.15)))
     )
@@
     (tags "resistor 0805")
     (attr smd)
-    (fp_text reference "" (at 0 -1.7 270) (layer F.SilkS)
+    (fp_text reference R1 (at 0 -1.7 270) (layer F.SilkS)
       (effects (font (size 1 1) (thickness 0.15)))
     )
@@
   )
   (module DQM_kicad_new:U.Fl_SMD (layer F.Cu)
-    (at 142.7 158.95)
+    (at 142.85 157.275)
     (fp_text reference "" (at -2.3 -0.7) (layer F.SilkS)
       (effects (font (size 1 1) (thickness 0.15)))
@@
     (fp_line (start 2.2 -1.9) (end 0 -1.9) (layer F.SilkS) (width 0.15))
     (pad 1 smd rect (at 1.1 0.6) (size 2.2 1) (layers F.Cu F.Paste F.Mask)
+      (net 15 GND))
+    (pad 1 smd rect (at 1.1 -2.5) (size 2.2 1) (layers F.Cu F.Paste F.Mask)
+      (net 15 GND))
+    (pad 2 smd rect (at 2.7 -1) (size 1.05 1) (layers F.Cu F.Paste F.Mask)
       (net 16 ANT))
-    (pad 1 smd rect (at 1.1 -2.5) (size 2.2 1) (layers F.Cu F.Paste F.Mask)
-      (net 16 ANT))
-    (pad 2 smd rect (at 2.7 -1) (size 1.05 1) (layers F.Cu F.Paste F.Mask)
-      (net 15 GND))
   )
   (module DQM_kicad_new:ArduProMini (layer F.Cu)
@@
       (net 23 NSS))
   )
+  (module Pin_Headers:Pin_Header_Straight_1x02_Pitch2.54mm (layer F.Cu)
+    (at 142.775 160.65 90)
+    (descr "Through hole straight pin header, 1x02, 2.54mm pitch, single row")
+    (tags "Through hole pin header THT 1x02 2.54mm single row")
+    (fp_text reference "" (at 0 -2.33 90) (layer F.SilkS)
+      (effects (font (size 1 1) (thickness 0.15)))
+    )
+    (fp_text value "" (at 0 4.87 90) (layer F.Fab)
+      (effects (font (size 1 1) (thickness 0.15)))
+    )
+    (fp_line (start -0.635 -1.27) (end 1.27 -1.27) (layer F.Fab) (width 0.1))
+    (fp_line (start 1.27 -1.27) (end 1.27 3.81) (layer F.Fab) (width 0.1))
+    (fp_line (start 1.27 3.81) (end -1.27 3.81) (layer F.Fab) (width 0.1))
+    (fp_line (start -1.27 3.81) (end -1.27 -0.635) (layer F.Fab) (width 0.1))
+    (fp_line (start -1.27 -0.635) (end -0.635 -1.27) (layer F.Fab) (width 0.1))
+    (fp_line (start -1.33 3.87) (end 1.33 3.87) (layer F.SilkS) (width 0.12))
+    (fp_line (start -1.33 1.27) (end -1.33 3.87) (layer F.SilkS) (width 0.12))
+    (fp_line (start 1.33 1.27) (end 1.33 3.87) (layer F.SilkS) (width 0.12))
+    (fp_line (start -1.33 1.27) (end 1.33 1.27) (layer F.SilkS) (width 0.12))
+    (fp_line (start -1.33 0) (end -1.33 -1.33) (layer F.SilkS) (width 0.12))
+    (fp_line (start -1.33 -1.33) (end 0 -1.33) (layer F.SilkS) (width 0.12))
+    (fp_line (start -1.8 -1.8) (end -1.8 4.35) (layer F.CrtYd) (width 0.05))
+    (fp_line (start -1.8 4.35) (end 1.8 4.35) (layer F.CrtYd) (width 0.05))
+    (fp_line (start 1.8 4.35) (end 1.8 -1.8) (layer F.CrtYd) (width 0.05))
+    (fp_line (start 1.8 -1.8) (end -1.8 -1.8) (layer F.CrtYd) (width 0.05))
+    (fp_text user %R (at 0 1.27 180) (layer F.Fab)
+      (effects (font (size 1 1) (thickness 0.15)))
+    )
+    (pad 1 thru_hole rect (at 0 0 90) (size 1.7 1.7) (drill 1) (layers *.Cu *.Mask)
+      (net 15 GND))
+    (pad 2 thru_hole oval (at 0 2.54 90) (size 1.7 1.7) (drill 1) (layers *.Cu *.Mask)
+      (net 16 ANT))
+    (model ${KISYS3DMOD}/Pin_Headers.3dshapes/Pin_Header_Straight_1x02_Pitch2.54mm.wrl
+      (at (xyz 0 0 0))
+      (scale (xyz 1 1 1))
+      (rotate (xyz 0 0 0))
+    )
+  )
+  (gr_text + (at 147.85 161.275) (layer F.SilkS)
+    (effects (font (size 1.5 1.5) (thickness 0.3)))
+  )
   (gr_line (start 140.875 99.975) (end 174.95 99.975) (angle 90) (layer Edge.Cuts) (width 0.15))
   (gr_line (start 174.95 162.525) (end 174.95 162.625) (angle 90) (layer Edge.Cuts) (width 0.15))
   (gr_line (start 140.825 162.525) (end 174.95 162.525) (angle 90) (layer Edge.Cuts) (width 0.15))
-  (gr_text Ant (at 145.075 154.5) (layer F.SilkS)
+  (gr_text Ant (at 147.25 154.125 270) (layer F.SilkS)
     (effects (font (size 1.5 1.5) (thickness 0.3)))
   )
@@
   (gr_line (start 140.95 162.4) (end 140.95 99.9) (angle 90) (layer Edge.Cuts) (width 0.15))
   (gr_line (start 175 100) (end 175 162.5) (angle 90) (layer Edge.Cuts) (width 0.15))
-  (gr_text "v1.0 August 2018\nD Q McDonald" (at 158.725 105.45) (layer F.SilkS)
+  (gr_text "v1.1 August 2018\nD Q McDonald" (at 158.725 105.45) (layer F.SilkS)
     (effects (font (size 1 1) (thickness 0.25)))
   )
@@
   (segment (start 171.55 116.55) (end 171.55 114.01) (width 0.5) (layer F.Cu) (net 14) (status 30))
   (segment (start 171.4972 116.55) (end 171.55 116.55) (width 0.5) (layer F.Cu) (net 14) (status 30))
-  (segment (start 145.4 157.95) (end 148.65 157.95) (width 0.5) (layer F.Cu) (net 15))
+  (segment (start 142.775 160.65) (end 142.775 159.05) (width 0.5) (layer F.Cu) (net 15) (status 400000))
+  (segment (start 142.775 159.05) (end 143.95 157.875) (width 0.5) (layer F.Cu) (net 15) (status 800000))
+  (segment (start 143.95 154.775) (end 143.95 154.175) (width 0.5) (layer F.Cu) (net 15) (status 400000))
+  (segment (start 143 153.225) (end 143 151.35) (width 0.5) (layer F.Cu) (net 15) (status 800000))
+  (segment (start 143.95 154.175) (end 143 153.225) (width 0.5) (layer F.Cu) (net 15))
   (segment (start 148.65 157.95) (end 148.8 158.1) (width 0.5) (layer F.Cu) (net 15))
   (segment (start 148.8 158.1) (end 148.8 155.55) (width 0.5) (layer F.Cu) (net 15))
@@
   (segment (start 146.9 117.55) (end 143.825 117.55) (width 0.5) (layer F.Cu) (net 15))
   (segment (start 148.3236 118.9736) (end 146.9 117.55) (width 0.5) (layer F.Cu) (net 15))
-  (segment (start 143.8 159.55) (end 142.025 159.55) (width 0.5) (layer F.Cu) (net 16))
-  (segment (start 142.125 156.85) (end 143.4 156.85) (width 0.5) (layer F.Cu) (net 16))
-  (segment (start 141.6 157.375) (end 142.125 156.85) (width 0.5) (layer F.Cu) (net 16))
-  (segment (start 141.6 159.125) (end 141.6 157.375) (width 0.5) (layer F.Cu) (net 16))
-  (segment (start 142.025 159.55) (end 141.6 159.125) (width 0.5) (layer F.Cu) (net 16))
-  (segment (start 143.4 156.85) (end 143.8 156.45) (width 0.5) (layer F.Cu) (net 16))
-  (segment (start 148.8 159.6) (end 143.8 159.55) (width 0.5) (layer F.Cu) (net 16) (status 20))
+  (segment (start 143.55 155.175) (end 143.95 154.775) (width 0.5) (layer F.Cu) (net 15) (status 30))
+  (segment (start 147.05 159.6) (end 146.365 159.6) (width 0.5) (layer F.Cu) (net 16))
+  (segment (start 146.365 159.6) (end 145.315 160.65) (width 0.5) (layer F.Cu) (net 16) (status 800000))
+  (segment (start 148.8 159.6) (end 147.05 159.6) (width 0.5) (layer F.Cu) (net 16))
+  (segment (start 147.05 159.6) (end 145.55 156.275) (width 0.5) (layer F.Cu) (net 16) (status 20))
   (segment (start 170.085 104.675) (end 169.3 104.675) (width 0.5) (layer F.Cu) (net 17))
   (segment (start 169.3 104.675) (end 166.2811 107.6939) (width 0.5) (layer F.Cu) (net 17))

Commit message: Antenna connection fix
Fixed error with antenna connections being shorted to ground
Other:
- board text added: "v1.2 May 2020 D Q McDonald"
- board text removed: "v1.1 August 2018 D Q McDonald"
Changed lines of the file:
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@@
-(kicad_pcb (version 4) (host pcbnew 4.0.7)
+(kicad_pcb (version 20171130) (host pcbnew "(5.1.2-1)-1")
   (general
-    (links 38)
-    (no_connects 0)
-    (area 140.749999 99.824999 175.075001 162.700001)
     (thickness 1.6)
     (drawings 27)
@@
     (zone_45_only no)
     (trace_min 0.2)
-    (segment_width 0.2)
-    (edge_width 0.15)
     (via_size 0.6)
     (via_drill 0.4)
@@
     (uvia_min_size 0.2)
     (uvia_min_drill 0.1)
+    (edge_width 0.15)
+    (segment_width 0.2)
     (pcb_text_width 0.3)
     (pcb_text_size 1.5 1.5)
@@
     (visible_elements FFFFFF7F)
     (pcbplotparams
-      (layerselection 0x010f0_80000001)
+      (layerselection 0x010f0_ffffffff)
       (usegerberextensions false)
+      (usegerberattributes false)
+      (usegerberadvancedattributes false)
+      (creategerberjobfile false)
       (excludeedgelayer true)
       (linewidth 0.100000)
@@
       (hpglpennumber 1)
       (hpglpenspeed 20)
-      (hpglpendiameter 15)
-      (hpglpenoverlay 2)
+      (hpglpendiameter 15.000000)
       (psnegative false)
       (psa4output false)
@@
       (drillshape 0)
       (scaleselection 1)
-      (outputdirectory Gerber/))
+      (outputdirectory "Gerber/"))
   )
   (net 0 "")
@@
     (fp_line (start 1.8 4.35) (end 1.8 -1.8) (layer F.CrtYd) (width 0.05))
     (fp_line (start 1.8 -1.8) (end -1.8 -1.8) (layer F.CrtYd) (width 0.05))
-    (fp_text user %R (at 0 1.27 360) (layer F.Fab)
+    (fp_text user %R (at 0 1.27) (layer F.Fab)
       (effects (font (size 1 1) (thickness 0.15)))
     )
@@
   (gr_line (start 140.95 162.4) (end 140.95 99.9) (angle 90) (layer Edge.Cuts) (width 0.15))
   (gr_line (start 175 100) (end 175 162.5) (angle 90) (layer Edge.Cuts) (width 0.15))
-  (gr_text "v1.1 August 2018\nD Q McDonald" (at 158.725 105.45) (layer F.SilkS)
+  (gr_text "v1.2 May 2020\nD Q McDonald" (at 158.725 105.45) (layer F.SilkS)
     (effects (font (size 1 1) (thickness 0.25)))
   )
@@
   (segment (start 171.55 116.55) (end 171.55 114.01) (width 0.5) (layer F.Cu) (net 14) (status 30))
   (segment (start 171.4972 116.55) (end 171.55 116.55) (width 0.5) (layer F.Cu) (net 14) (status 30))
-  (segment (start 142.775 160.65) (end 142.775 159.05) (width 0.5) (layer F.Cu) (net 15) (status 400000))
-  (segment (start 142.775 159.05) (end 143.95 157.875) (width 0.5) (layer F.Cu) (net 15) (status 800000))
-  (segment (start 143.95 154.775) (end 143.95 154.175) (width 0.5) (layer F.Cu) (net 15) (status 400000))
-  (segment (start 143 153.225) (end 143 151.35) (width 0.5) (layer F.Cu) (net 15) (status 800000))
+  (segment (start 142.775 160.65) (end 142.775 159.05) (width 0.5) (layer F.Cu) (net 15))
+  (segment (start 142.775 159.05) (end 143.95 157.875) (width 0.5) (layer F.Cu) (net 15))
+  (segment (start 143.95 154.775) (end 143.95 154.175) (width 0.5) (layer F.Cu) (net 15))
+  (segment (start 143 153.225) (end 143 151.35) (width 0.5) (layer F.Cu) (net 15))
   (segment (start 143.95 154.175) (end 143 153.225) (width 0.5) (layer F.Cu) (net 15))
   (segment (start 148.65 157.95) (end 148.8 158.1) (width 0.5) (layer F.Cu) (net 15))
@@
   (segment (start 143.55 155.175) (end 143.95 154.775) (width 0.5) (layer F.Cu) (net 15) (status 30))
   (segment (start 147.05 159.6) (end 146.365 159.6) (width 0.5) (layer F.Cu) (net 16))
-  (segment (start 146.365 159.6) (end 145.315 160.65) (width 0.5) (layer F.Cu) (net 16) (status 800000))
+  (segment (start 146.365 159.6) (end 145.315 160.65) (width 0.5) (layer F.Cu) (net 16))
   (segment (start 148.8 159.6) (end 147.05 159.6) (width 0.5) (layer F.Cu) (net 16))
   (segment (start 147.05 159.6) (end 145.55 156.275) (width 0.5) (layer F.Cu) (net 16) (status 20))

Commit message: Updated Kicad
Parts:
- added 1uF: C, Capacitors_SMD:C_0805_HandSoldering, F.Cu at (152.2, 104.4)
- added 1uF: C, Capacitors_SMD:C_0805_HandSoldering, F.Cu at (165.2, 105.0)
- added U2: MCP1703A, TO_SOT_Packages_SMD:SOT-223-3_TabPin2, F.Cu at (158.7, 106.0)
- K1: renamed from ?; value (none) -> CONN_3
- P1: renamed from ?; value (none) -> CONN_5
- P2, P3: renamed from ?; value (none) -> CONN_4
- P4, P5, P6: renamed from ?; value (none) -> CONN_2
- SW1: renamed from ?; value (none) -> SPST
Connections:
- P5 pad 2: Vin -> Net-(C1-Pad1)
- uP1 pad 19: Vin -> Net-(uP1-Pad19)
Routing:
- net Net-(C1-Pad1): track 0.00 -> 37.1 mm
- net GND: track 98.5 -> 128.0 mm
- net V3.3: track 41.7 -> 57.3 mm
- net Vin: track 8.71 -> 0.00 mm
Other:
- board size 34.2 x 62.7 mm -> 34.1 x 62.8 mm
- net class Default removed
- board text added: "v1.3 June 2020 D Q McDonald"
- board text removed: "v1.2 May 2020 D Q McDonald"
